File: DC.kicad_sch (KiCad schematic)
At the start: 5 parts, among them U1 LT8610, U2 LT3483AxS6, U3 LT3094xMSE, U4 ADP7118ACPZN, U5 ADP7118ACPZN

Commit message: DC almost done
Parts:
- added C1: 100nF, SparkFun-Resistor:R_0603_1608Metric, symbol Device:C
- added C2: 10pF, SparkFun-Resistor:R_0603_1608Metric, symbol Device:C
- added C3: C, symbol Device:C
- added C4: 1uF, symbol Device:C
- added L1: L, symbol Device:L
- added R1, R2, R3: 1k, SparkFun-Resistor:R_0603_1608Metric, symbol SparkFun:R
Connections:
- net GND: now reaches U1.1 (SYNC)
- net GND: now also U1.17 (GND), U1.7 (PGND), U1.8 (PGND), C3.2, C4.2, R1.2, R3.2
- net at U1.10 (SW): now also U1.11 (SW), U1.9 (SW), C1.2, L1.1
- net at U1.12 (BST): now also C1.1
- net at U1.13 (INTVCC): now also C4.1
- net at U1.14 (BIAS): now also C2.2, L1.2, R2.1
- net at U1.16 (FB): now also C2.1, R2.2, R3.1
- net at U1.3 (RT): now also C3.1, R1.1
- net at U1.4 (EN/UV): now also U1.5 (VIN), U1.6 (VIN)
- no-connect marks 0 -> 1
Other:
- moved on the sheet: U1

Commit message: final before push to master
Parts:
- added C10, C11, C12, C13, C14, C15, C6, C7, C8, C9: C, SparkFun-Resistor:R_0603_1608Metric, symbol Device:C
- added C5: C, symbol Device:C
- added D1: ${DEVICE}, Diode_THT:D_DO-35_SOD27_P7.62mm_Horizontal, symbol CERN:Diode Schottky
- added L2: L, symbol Device:L
- added R10, R11, R12, R13, R4, R5, R6, R7, R8, R9: 1k, SparkFun-Resistor:R_0603_1608Metric, symbol SparkFun:R
Connections:
- net GND: now also U2.2 (GND), U3.9 (GND), U4.3 (GND), U4.7 (GND), U5.3 (GND), U5.7 (GND), C10.2, C11.2, C12.2, C13.2, C14.2, C15.2, C7.2, C8.2, C9.2, R11.2, R13.2, R7.2, R8.2, R9.2
- net at R1.1, U1.3 (RT): no longer C3.1
- net at C2.2, L1.2, R2.1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: now also U4.4 (EN), U4.6 (VIN), U5.4 (EN), U5.6 (VIN), C12.1, C14.1
- net at U1.4 (EN/UV), U1.5 (VIN), U1.6 (VIN): now also C3.1, U2.4 (~{SHDN}), U2.6 (V_{IN}), C7.1, L2.1
- net at U2.3 (FB): now also C6.2, R5.2
- net at U2.5 (D): now also C5.2, D1.1 (C)
- net at U4.1 (VOUT): now also C13.1, R10.1
- net at U4.2 (SENSE/ADJ): now also R10.2, R11.1
- net at U5.1 (VOUT): now also C15.1, R12.1
- net at U5.2 (SENSE/ADJ): now also R12.2, R13.1
- net at U3.1 (IN), U3.13 (IN), U3.2 (IN): now also U3.3 (EN/UV), C10.1, C6.1, C8.1, R4.2, R5.1
- net at U3.10 (OUTS): now also U3.11 (OUT), U3.12 (OUT), C11.1, R6.1
- net at U3.5 (PGFB): now also R6.2, R7.1
- net at U3.6 (ILIM): now also R8.1
- net at U3.8 (SET): now also C9.1, R9.1
- new net: C5.1, L2.2
- new net: D1.2 (A), R4.1
- no-connect marks 1 -> 4
Other:
- moved on the sheet: C3, U3

Commit message: some minor changes to DC
Parts:
- removed R6, R7, R8: 1k, SparkFun-Resistor:R_0603_1608Metric, symbol SparkFun:R
- C13, C15: value C -> 2.2uF
- L1: value L -> 6.2uH
- R1: value 1k -> 33.2k
- R10, R2: value 1k -> 5.1k
- R11: value 1k -> 1.6k
- R12: value 1k -> 8.2k
- R13: value 1k -> 4.7k
- R3: value 1k -> 820
- R8: renamed from R9; value 1k -> 50k
Connections:
- net at U3.5 (PGFB): now also C10.1, C6.1, C8.1, R4.2, R5.1, U3.1 (IN), U3.13 (IN), U3.2 (IN), U3.3 (EN/UV)
- no-connect marks 4 -> 7
